File: pcb/breakout_board_v2/breakout_board_v2.kicad_pcb (KiCad board)
At the start: 4 copper layers, 81.3 x 41.9 mm, 61 parts, among them J1 HKSPI_HDR, J2 SMA_CONN, J3 GPIO_HDR, SW1 DSHP08TSGER, U1 caravel-M.2-card, U2 DNF, U3 AP2112K-1.8, U4 74HC4050, U5 74HC4050

Commit message: cleanup boards
Parts:
- added REF**: OSHW-Logo_5.7x6mm_SilkScreen, Symbol:OSHW-Logo_5.7x6mm_SilkScreen, F.Cu at (240.5, 95.0)
