File: pcb/breakout_board_v1/breakout_board_v1.kicad_pcb (KiCad board)
At the start: 4 copper layers, 81.3 x 41.9 mm, 45 parts, among them J1 HKSPI_HDR, J2 SMA_CONN, J3 GPIO_HDR, SW1 DSHP08TSGER, U1 caravel-M.2-card, U2 DNF, U3 AP2112K-1.8

Commit message: cleanup boards
Parts:
- moved REF** 0.66 mm to (248.9, 90.8)
Routing:
- net GND: track 93.0 -> 93.1 mm, vias 49 -> 151
